File: pcb/imu/imu.kicad_sch (KiCad schematic)
At the start: 5 parts

Commit message: update pcb
Parts:
- J1: renamed from J?; footprint (none) -> Connector_JST:JST_ZE_BM06B-ZESS-TBT_1x06-1MP_P1.50mm_Vertical
- gave numbers to parts that had none: 4
Changed lines of the file:
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@@
   (symbol (lib_id "power:GND") (at 110.49 107.95 0) (mirror y) (unit 1)
     (in_bom yes) (on_board yes)
-    (property "Reference" "#PWR?" (id 0) (at 110.49 114.3 0)
+    (property "Reference" "#PWR0103" (id 0) (at 110.49 114.3 0)
       (effects (font (size 1.27 1.27)) hide)
     )
@@
   (symbol (lib_id "power:GND") (at 115.57 107.95 0) (mirror y) (unit 1)
     (in_bom yes) (on_board yes)
-    (property "Reference" "#PWR?" (id 0) (at 115.57 114.3 0)
+    (property "Reference" "#PWR0102" (id 0) (at 115.57 114.3 0)
       (effects (font (size 1.27 1.27)) hide)
     )
@@
   (symbol (lib_id "power:+3.3V") (at 90.17 80.01 0) (unit 1)
     (in_bom yes) (on_board yes)
-    (property "Reference" "#PWR?" (id 0) (at 90.17 83.82 0)
+    (property "Reference" "#PWR0101" (id 0) (at 90.17 83.82 0)
       (effects (font (size 1.27 1.27)) hide)
     )
@@
   (symbol (lib_id "Device:C_Small") (at 90.17 87.63 0) (unit 1)
     (in_bom yes) (on_board yes)
-    (property "Reference" "C?" (id 0) (at 83.82 86.36 0)
+    (property "Reference" "C1" (id 0) (at 83.82 86.36 0)
       (effects (font (size 1.27 1.27)) (justify left))
     )
@@
   (symbol (lib_id "Device:C_Small") (at 110.49 93.98 0) (unit 1)
     (in_bom yes) (on_board yes)
-    (property "Reference" "C?" (id 0) (at 106.68 92.71 0)
+    (property "Reference" "C3" (id 0) (at 106.68 92.71 0)
       (effects (font (size 1.27 1.27)) (justify left))
     )
@@
   (symbol (lib_id "power:+3.3V") (at 189.23 81.28 0) (unit 1)
     (in_bom yes) (on_board yes)
-    (property "Reference" "#PWR?" (id 0) (at 189.23 85.09 0)
+    (property "Reference" "#PWR0108" (id 0) (at 189.23 85.09 0)
       (effects (font (size 1.27 1.27)) hide)
     )
@@
   (symbol (lib_id "My_Device:MPU-6500") (at 123.19 85.09 0) (unit 1)
     (in_bom yes) (on_board yes)
-    (property "Reference" "U?" (id 0) (at 133.985 78.359 0))
+    (property "Reference" "U1" (id 0) (at 133.985 78.359 0))
     (property "Value" "MPU-6500" (id 1) (at 133.985 80.6704 0))
     (property "Footprint" "Package_DFN_QFN:QFN-24-1EP_3x3mm_P0.4mm_EP1.75x1.6mm" (id 2) (at 133.35 80.01 0)
@@
   (symbol (lib_id "power:+3.3V") (at 115.57 80.01 0) (unit 1)
     (in_bom yes) (on_board yes)
-    (property "Reference" "#PWR?" (id 0) (at 115.57 83.82 0)
+    (property "Reference" "#PWR0106" (id 0) (at 115.57 83.82 0)
       (effects (font (size 1.27 1.27)) hide)
     )
@@
   (symbol (lib_id "power:GND") (at 90.17 96.52 0) (mirror y) (unit 1)
     (in_bom yes) (on_board yes)
-    (property "Reference" "#PWR?" (id 0) (at 90.17 102.87 0)
+    (property "Reference" "#PWR0105" (id 0) (at 90.17 102.87 0)
       (effects (font (size 1.27 1.27)) hide)
     )
@@
   (symbol (lib_id "power:GND") (at 151.13 107.95 0) (mirror y) (unit 1)
     (in_bom yes) (on_board yes)
-    (property "Reference" "#PWR?" (id 0) (at 151.13 114.3 0)
+    (property "Reference" "#PWR0109" (id 0) (at 151.13 114.3 0)
       (effects (font (size 1.27 1.27)) hide)
     )
@@
   (symbol (lib_id "Connector:Conn_01x06_Female") (at 199.39 88.9 0) (unit 1)
     (in_bom yes) (on_board yes) (fields_autoplaced)
-    (property "Reference" "J?" (id 0) (at 200.66 88.8999 0)
+    (property "Reference" "J1" (id 0) (at 200.66 88.8999 0)
       (effects (font (size 1.27 1.27)) (justify left))
     )
@@
       (effects (font (size 1.27 1.27)) (justify left))
     )
-    (property "Footprint" "" (id 2) (at 199.39 88.9 0)
+    (property "Footprint" "Connector_JST:JST_ZE_BM06B-ZESS-TBT_1x06-1MP_P1.50mm_Vertical" (id 2) (at 199.39 88.9 0)
       (effects (font (size 1.27 1.27)) hide)
     )
@@
   (symbol (lib_id "power:GND") (at 120.65 107.95 0) (mirror y) (unit 1)
     (in_bom yes) (on_board yes)
-    (property "Reference" "#PWR?" (id 0) (at 120.65 114.3 0)
+    (property "Reference" "#PWR0104" (id 0) (at 120.65 114.3 0)
       (effects (font (size 1.27 1.27)) hide)
     )
@@
   (symbol (lib_id "Device:C_Small") (at 99.06 87.63 0) (unit 1)
     (in_bom yes) (on_board yes)
-    (property "Reference" "C?" (id 0) (at 92.71 86.36 0)
+    (property "Reference" "C2" (id 0) (at 92.71 86.36 0)
       (effects (font (size 1.27 1.27)) (justify left))
     )
@@
   (symbol (lib_id "power:GND") (at 189.23 101.6 0) (mirror y) (unit 1)
     (in_bom yes) (on_board yes)
-    (property "Reference" "#PWR?" (id 0) (at 189.23 107.95 0)
+    (property "Reference" "#PWR0107" (id 0) (at 189.23 107.95 0)
       (effects (font (size 1.27 1.27)) hide)
     )
@@
   )
   (symbol_instances
+    (path "/4046dc24-7a91-4e8d-8122-a057188bf243"
+      (reference "#PWR0101") (unit 1) (value "+3.3V") (footprint "")
+    )
+    (path "/3a180575-7980-4970-b8e1-3c4f49f39811"
+      (reference "#PWR0102") (unit 1) (value "GND") (footprint "")
+    )
     (path "/24757894-f9c3-4246-a6be-978b7e0ba1b9"
-      (reference "#PWR?") (unit 1) (value "GND") (footprint "")
-    )
-    (path "/3a180575-7980-4970-b8e1-3c4f49f39811"
-      (reference "#PWR?") (unit 1) (value "GND") (footprint "")
-    )
-    (path "/4046dc24-7a91-4e8d-8122-a057188bf243"
-      (reference "#PWR?") (unit 1) (value "+3.3V") (footprint "")
+      (reference "#PWR0103") (unit 1) (value "GND") (footprint "")
+    )
+    (path "/dcf2818c-0257-47dd-ac6e-5966a20d99ad"
+      (reference "#PWR0104") (unit 1) (value "GND") (footprint "")
+    )
+    (path "/a08efb6e-b616-4aff-ad65-0c2fc809716a"
+      (reference "#PWR0105") (unit 1) (value "GND") (footprint "")
+    )
+    (path "/9a16068a-d492-4ddd-a324-01fdaf34caea"
+      (reference "#PWR0106") (unit 1) (value "+3.3V") (footprint "")
+    )
+    (path "/f6226537-5216-468f-b096-85abb467e18b"
+      (reference "#PWR0107") (unit 1) (value "GND") (footprint "")
     )
     (path "/70674246-a080-4cd6-961f-c56b78656b79"
-      (reference "#PWR?") (unit 1) (value "+3.3V") (footprint "")
-    )
-    (path "/9a16068a-d492-4ddd-a324-01fdaf34caea"
-      (reference "#PWR?") (unit 1) (value "+3.3V") (footprint "")
-    )
-    (path "/a08efb6e-b616-4aff-ad65-0c2fc809716a"
-      (reference "#PWR?") (unit 1) (value "GND") (footprint "")
+      (reference "#PWR0108") (unit 1) (value "+3.3V") (footprint "")
     )
     (path "/bbb4b41d-6217-4f2c-a089-c167cba2a65b"
-      (reference "#PWR?") (unit 1) (value "GND") (footprint "")
-    )
-    (path "/dcf2818c-0257-47dd-ac6e-5966a20d99ad"
-      (reference "#PWR?") (unit 1) (value "GND") (footprint "")
-    )
-    (path "/f6226537-5216-468f-b096-85abb467e18b"
-      (reference "#PWR?") (unit 1) (value "GND") (footprint "")
+      (reference "#PWR0109") (unit 1) (value "GND") (footprint "")
     )
     (path "/4f45cac2-0970-4321-b8ca-ae4d227693ef"
-      (reference "C?") (unit 1) (value "0.1u") (footprint "Capacitor_SMD:C_0603_1608Metric_Pad1.08x0.95mm_HandSolder")
+      (reference "C1") (unit 1) (value "0.1u") (footprint "Capacitor_SMD:C_0603_1608Metric_Pad1.08x0.95mm_HandSolder")
+    )
+    (path "/ddd16aa2-2f29-4cdb-8f5c-ec1b09797e97"
+      (reference "C2") (unit 1) (value "0.1u") (footprint "Capacitor_SMD:C_0603_1608Metric_Pad1.08x0.95mm_HandSolder")
     )
     (path "/62da50b5-05e3-4bf7-9e1b-a1f56778e9b2"
-      (reference "C?") (unit 1) (value "0.1u") (footprint "Capacitor_SMD:C_0603_1608Metric_Pad1.08x0.95mm_HandSolder")
-    )
-    (path "/ddd16aa2-2f29-4cdb-8f5c-ec1b09797e97"
-      (reference "C?") (unit 1) (value "0.1u") (footprint "Capacitor_SMD:C_0603_1608Metric_Pad1.08x0.95mm_HandSolder")
+      (reference "C3") (unit 1) (value "0.1u") (footprint "Capacitor_SMD:C_0603_1608Metric_Pad1.08x0.95mm_HandSolder")
     )
     (path "/ce3ab929-8030-43a7-b629-0647da722a42"
-      (reference "J?") (unit 1) (value "Conn_01x06_Female") (footprint "")
+      (reference "J1") (unit 1) (value "Conn_01x06_Female") (footprint "Connector_JST:JST_ZE_BM06B-ZESS-TBT_1x06-1MP_P1.50mm_Vertical")
     )
     (path "/73570ede-ff60-41ff-a5a0-1cb3b70c8474"
-      (reference "U?") (unit 1) (value "MPU-6500") (footprint "Package_DFN_QFN:QFN-24-1EP_3x3mm_P0.4mm_EP1.75x1.6mm")
-    )
-  )
+      (reference "U1") (unit 1) (value "MPU-6500") (footprint "Package_DFN_QFN:QFN-24-1EP_3x3mm_P0.4mm_EP1.75x1.6mm")
+    )
+  )
