File: pcb/motor_driver/user_interface.kicad_sch (KiCad schematic)
At the start: 14 parts

Commit message: update pcb
Parts:
- removed C?: 0.1u, Capacitor_SMD:C_0201_0603Metric, symbol Device:C_Small
- removed D?: LED4, LED_SMD:LED_0402_1005Metric, symbol Device:LED
- removed D?: LED2, LED_SMD:LED_0402_1005Metric, symbol Device:LED
- removed D?: LED3, LED_SMD:LED_0402_1005Metric, symbol Device:LED
- removed D?: LED1, LED_SMD:LED_0402_1005Metric, symbol Device:LED
- removed Q?: BSS138, Package_TO_SOT_SMD:SOT-23, symbol Transistor_FET:BSS138
- removed R? (x4): 1k, Resistor_SMD:R_0201_0603Metric, symbol Device:R_Small
- removed R?: 10k, Resistor_SMD:R_0201_0603Metric, symbol Device:R_Small
- removed R?: 100k, Resistor_SMD:R_0201_0603Metric, symbol Device:R_Small
- removed SP?: SMT-0440, omni:STM0440-T-R, symbol My_Device:SMT-0440
- removed SW?: TVAF06-A020B-R, half_mouse_lib:TVAF06-A020B-R, symbol My_Device:SKRPACE
