File: pcb/motor_driver/motor_driver.kicad_pcb (KiCad board)
At the start: 2 copper layers, 99 parts, among them J1 XT60PW-M, J2 1-84953-1, J3 Conn_ARM_JTAG_SWD_10, J4 UART1 SH, J5 Conn, Q1 BSS138, SW1 SKRPACE010, SW2 SKRPACE010, U1 USBLC6-4SC6, U10 STM32G431CB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

Commit message: delete ESD protection
Parts:
- removed C37, C38, C6: 0.1u, Capacitor_SMD:C_0603_1608Metric_Pad1.08x0.95mm_HandSolder
- removed U11, U13, U2: USBLC6-4SC6, Package_TO_SOT_SMD:SOT-23-6

Commit message: update pcb
Parts:
- removed C31, C32: 0.1u, Capacitor_SMD:C_0201_0603Metric
- removed C35: 1u, Capacitor_SMD:C_0201_0603Metric
- added ?: , , F.Cu at (114.4, 97.8)
- added ?: , , F.Cu at (91.9, 97.8)
- added ?: , , F.Cu at (113.8, 97.0)
- added ?: , , F.Cu at (91.4, 97.0)
- added ?: , , F.Cu at (103.9, 96.2)
- added ?: , , F.Cu at (103.9, 97.8)
- added ?: , , F.Cu at (103.4, 97.0)
- added ?: , , F.Cu at (92.9, 97.8)
- added ?: , , F.Cu at (113.3, 97.8)
- added ?: , , F.Cu at (91.9, 96.2)
- added ?: , , F.Cu at (102.5, 97.0)
- added ?: , , F.Cu at (102.9, 97.8)
- added ?: , , F.Cu at (104.4, 97.0)
- added ?: , , F.Cu at (114.4, 96.2)
- added ?: , , F.Cu at (114.8, 97.0)
- added ?: , , F.Cu at (92.9, 96.2)
- added ?: , , F.Cu at (103.0, 96.2)
- added ?: , , F.Cu at (113.4, 96.2)
- added ?: , , F.Cu at (93.4, 97.0)
- added ?: , , F.Cu at (112.9, 97.0)
- added ?: , , F.Cu at (92.4, 97.0)
- C1, C14, C15, C16, C17, C18, C19, C2, C25, C3, C33, C36, C4, C5, C7, C9: footprint Capacitor_SMD:C_0603_1608Metric_Pad1.08x0.95mm_HandSolder -> Capacitor_SMD:C_0603_1608Metric
- C22, C23, C24, C26, C28: footprint Capacitor_SMD:C_0402_1005Metric -> Capacitor_SMD:C_0603_1608Metric
- C27, C29, C30: footprint Capacitor_SMD:C_0201_0603Metric -> Capacitor_SMD:C_0603_1608Metric
- C34: value 0.01u -> 0.1u; footprint Capacitor_SMD:C_0402_1005Metric -> Capacitor_SMD:C_0603_1608Metric
- D4: footprint LED_SMD:LED_0603_1608Metric_Pad1.05x0.95mm_HandSolder -> LED_SMD:LED_0402_1005Metric
- J1: footprint bldc_lib:XT60PWM -> Connector_AMASS:AMASS_XT30U-F_1x02_P5.0mm_Vertical
- R13: footprint Resistor_SMD:R_0402_1005Metric_Pad0.72x0.64mm_HandSolder -> Resistor_SMD:R_0603_1608Metric_Pad0.98x0.95mm_HandSolder
- R20, R22, R23, R24, R25: footprint Resistor_SMD:R_0201_0603Metric -> Resistor_SMD:R_0603_1608Metric
- R26, U12: moved to F.Cu
- SW1: value SKRPACE010 -> RESET
- SW2: value SKRPACE010 -> USER
- U3: footprint Package_DFN_QFN:QFN-40-1EP_6x6mm_P0.5mm_EP4.6x4.6mm_ThermalVias -> Package_DFN_QFN:QFN-40-1EP_6x6mm_P0.5mm_EP4.6x4.6mm
- moved C34 70.2 mm to (130.8, 119.1), turned to -90 degrees
- moved C27 56.7 mm to (123.9, 103.5), turned to 90 degrees
- moved C26 55.0 mm to (123.3, 106.2), turned to 180 degrees
- moved C29 54.1 mm to (133.3, 115.3)
- moved C30 53.3 mm to (133.2, 105.7), turned to 90 degrees
- moved D4 45.2 mm to (131.1, 127.4), turned to -90 degrees
- moved R3 42.0 mm to (92.0, 102.1)
- moved D3 41.9 mm to (92.0, 105.1)
- moved R2 41.1 mm to (94.9, 102.1)
- moved D2 41.0 mm to (94.9, 105.1)
- moved R1 40.3 mm to (97.7, 102.1)
- moved D1 40.3 mm to (97.7, 105.1)
- moved R13 39.3 mm to (131.1, 124.4), turned to 90 degrees
- moved R19 21.7 mm to (127.2, 97.2), turned to 90 degrees
- moved C1 21.3 mm to (106.5, 117.8)
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- renumbered U5 to Q2, U6 to Q3, U7 to Q4
Connections:
- J5 pad 2: /stm32g431cb/CAN_H -> /stm32g431cb/CAN_L
- J5 pad 3: /stm32g431cb/CAN_L -> /stm32g431cb/CAN_H
- SW1 pad 2: /stm32g431cb/RST_SW_ESD -> unconnected-(SW1-Pad2)
- U10 pad 11: /stm32g431cb/LED1 -> /stm32g431cb/DRV_CAL
- U10 pad 12: /stm32g431cb/LED2 -> /stm32g431cb/INLX
- U10 pad 13: /stm32g431cb/SPI1_SCK -> /drv8323/SPI1_CLK
- U10 pad 16: /drv8323/SS_ENC -> /stm32g431cb/SW1
- U10 pad 17: /stm32g431cb/SS_DRV -> /stm32g431cb/LED1
- U10 pad 18: unconnected-(U10-Pad18) -> /stm32g431cb/LED2
- U10 pad 2: /stm32g431cb/FAULTB -> /stm32g431cb/DRV_ENABLE
- U10 pad 22: /drv8323/INHC -> /stm32g431cb/LED3
- U10 pad 25: /stm32g431cb/SW1 -> /stm32g431cb/LED4
- U10 pad 26: /stm32g431cb/LED_CAN_TX -> unconnected-(U10-Pad26)
- U10 pad 27: /stm32g431cb/LED_CAN_RX -> unconnected-(U10-Pad27)
- U10 pad 29: unconnected-(U10-Pad29) -> /stm32g431cb/LED_CAN_RX
- U10 pad 3: /stm32g431cb/DRV_ENABLE -> /stm32g431cb/FAULTB
- U10 pad 30: /stm32g431cb/INLX -> /stm32g431cb/LED_CAN_TX
- U10 pad 39: /drv8323/INHA -> /drv8323/HALL_W
- U10 pad 4: /stm32g431cb/DRV_CAL -> /stm32g431cb/SS_DRV
- U10 pad 40: /drv8323/INHB -> /drv8323/HALL_U
- U10 pad 41: /drv8323/HALL_W -> /drv8323/HALL_V
- U10 pad 42: /drv8323/HALL_V -> /drv8323/SS_ENC
- U10 pad 43: /drv8323/HALL_U -> /drv8323/INHA
- U10 pad 44: /stm32g431cb/LED4 -> /drv8323/INHB
- U10 pad 46: /stm32g431cb/LED3 -> /drv8323/INHC
- U3 pad 21: /stm32g431cb/ADC1_3 -> /stm32g431cb/ADC1_1
- U3 pad 23: /stm32g431cb/ADC1_1 -> /stm32g431cb/ADC1_3
Routing:
- net GND: track 0.00 -> 354.4 mm, vias 0 -> 50
- net +5V: track 0.00 -> 70.3 mm, vias 0 -> 1
- net /drv8323/SPI1_MISO: track 0.00 -> 67.0 mm, vias 0 -> 3
- net /drv8323/SPI1_MOSI: track 0.00 -> 64.9 mm, vias 0 -> 3
- net /stm32g431cb/NRST: track 0.00 -> 61.4 mm, vias 0 -> 1
- net /drv8323/SPI1_CLK: track 0.00 -> 59.9 mm, vias 0 -> 3
- net /drv8323/SHA: track 0.00 -> 56.6 mm, vias 0 -> 2
- net /stm32g431cb/SS_DRV: track 0.00 -> 50.3 mm, vias 0 -> 2
- net /drv8323/SHC: track 0.00 -> 48.6 mm, vias 0 -> 2
- net +3.3V: track 0.00 -> 46.9 mm
- net /stm32g431cb/DRV_ENABLE: track 0.00 -> 46.8 mm, vias 0 -> 2
- net /drv8323/GHA: track 0.00 -> 43.5 mm, vias 0 -> 1
- net /drv8323/HALL_V: track 0.00 -> 42.8 mm, vias 0 -> 3
- net /drv8323/HALL_U: track 0.00 -> 39.4 mm, vias 0 -> 3
- net +3.3VA: track 0.00 -> 38.7 mm, vias 0 -> 2
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Other:
- board outline added: 55 x 55 mm
- copper layers 2 -> 4

Commit message: chore: add circuit git changes
Parts:
- removed ? (x21): , 
- C7: footprint Capacitor_SMD:C_0603_1608Metric -> Capacitor_SMD:C_0402_1005Metric
- moved C9 20.1 mm to (91.1, 91.7), turned to 90 degrees
- moved D1 14.5 mm to (99.7, 119.4)
- moved R1 14.5 mm to (99.7, 116.4)
- moved D2 14.5 mm to (96.8, 119.4)
- moved D3 14.5 mm to (93.9, 119.5)
- moved R2 14.5 mm to (96.8, 116.5)
- moved R3 14.5 mm to (93.9, 116.5)
- moved C8 10.5 mm to (95.3, 105.8), turned to -90 degrees
- moved C16 2.11 mm to (137.9, 83.6), turned to 90 degrees
- moved J1 0.79 mm to (102.6, 124.7)
- moved R26 0.57 mm to (127.8, 85.7)
- moved C7 0.43 mm to (113.5, 99.4)
- moved C26 0.10 mm to (123.3, 106.1)
Connections:
- U3 pad 41: (no net) -> GND
- U4 pad 15: (no net) -> GND
Routing:
- net GND: track 354.4 -> 1047.2 mm, vias 50 -> 106
- net /drv8323/INHA: track 7.53 -> 76.4 mm, vias 0 -> 2
- net /drv8323/INHB: track 10.8 -> 71.8 mm, vias 0 -> 2
- net /drv8323/INHC: track 14.8 -> 61.4 mm, vias 0 -> 2
- net +3.3V: track 46.9 -> 89.1 mm, vias 0 -> 5
- net +3.3VA: track 38.7 -> 76.0 mm, vias 2 -> 3
- net +5V: track 70.3 -> 38.9 mm, vias 1 -> 6
- net /stm32g431cb/NRST: track 61.4 -> 76.7 mm
- net +BATT: track 14.7 -> 11.6 mm, vias 0 -> 39
- net /stm32g431cb/LED_CAN_RX: track 22.4 -> 20.9 mm
- net /drv8323/SLB: track 31.8 -> 30.7 mm
- net /stm32g431cb/DRV_ENABLE: track 46.8 -> 45.7 mm
- net /stm32g431cb/LED_CAN_TX: track 20.1 -> 19.2 mm
- net /stm32g431cb/SW1: track 19.5 -> 18.7 mm
- net /drv8323/SLC: track 27.6 -> 28.3 mm
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- added copper zone on In2.Cu, net +3.3V
- added copper zone on In2.Cu, net +5V
- added copper zone on In2.Cu, net +BATT
- added copper zone on In1.Cu, net GND
- added copper zone on In2.Cu, net GND

Commit message: feat: fix most bug
Parts:
- removed J4: UART1 SH, Connector_PinHeader_2.54mm:PinHeader_1x04_P2.54mm_Vertical
- added H1: MountingHole, MountingHole:MountingHole_3.2mm_M3_Pad_TopBottom, F.Cu at (94.5, 79.3)
- added H2: MountingHole, MountingHole:MountingHole_3.2mm_M3_Pad_TopBottom, F.Cu at (94.5, 121.3)
- added H3: MountingHole, MountingHole:MountingHole_3.2mm_M3_Pad_TopBottom, F.Cu at (136.5, 79.3)
- added H4: MountingHole, MountingHole:MountingHole_3.2mm_M3_Pad_TopBottom, F.Cu at (136.5, 121.3)
- C14, C15, C16, C17, C18, C19, Q1, R20, SP1, U8, U9: moved to B.Cu
- moved C13 24.9 mm to (121.7, 98.8), turned to 0 degrees
- moved R6 23.5 mm to (115.3, 91.6)
- moved Q4 23.5 mm to (119.8, 91.2)
- moved R12 23.5 mm to (124.3, 91.6)
- moved R9 23.1 mm to (119.9, 96.5), turned to 180 degrees
- moved R7 20.1 mm to (98.1, 96.5)
- moved R4 20.1 mm to (93.6, 91.6)
- moved Q2 20.1 mm to (97.8, 91.2)
- moved R10 20.1 mm to (102.4, 91.6)
- moved C11 18.5 mm to (99.9, 98.7)
- moved R3 14.1 mm to (106.3, 123.2), turned to -90 degrees
- moved C5 12.9 mm to (103.6, 78.9), turned to -90 degrees
- moved D3 12.4 mm to (106.3, 120.2), turned to 90 degrees
- moved J1 11.5 mm to (98.7, 113.9)
- moved SP1 9.85 mm to (133.8, 121.3), turned to 90 degrees
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Connections:
- J2 pad 1: +5V -> /drv8323/SHC
- J2 pad 10: /drv8323/SHC -> /drv8323/HALL_W
- J2 pad 11: /drv8323/SHC -> +5V
- J2 pad 2: /drv8323/HALL_W -> /drv8323/SHC
- J2 pad 3: /drv8323/HALL_U -> /drv8323/SHB
- J2 pad 4: /drv8323/HALL_V -> /drv8323/SHB
- J2 pad 5: GND -> /drv8323/SHA
- J2 pad 7: /drv8323/SHA -> GND
- J2 pad 8: /drv8323/SHB -> /drv8323/HALL_V
- J2 pad 9: /drv8323/SHB -> /drv8323/HALL_U
- U10 pad 2: /stm32g431cb/DRV_ENABLE -> /stm32g431cb/FAULTB
- U10 pad 26: unconnected-(U10-Pad26) -> /stm32g431cb/LED_CAN_RX
- U10 pad 27: unconnected-(U10-Pad27) -> /drv8323/SPI2_CLK
- U10 pad 29: /stm32g431cb/LED_CAN_RX -> /drv8323/SPI2_MOSI
- U10 pad 3: /stm32g431cb/FAULTB -> /stm32g431cb/SS_DRV
- U10 pad 31: /stm32g431cb/USART1_TX -> unconnected-(U10-Pad31)
- U10 pad 32: /stm32g431cb/USART1_RX -> /drv8323/SPI2_MISO
- U10 pad 39: /drv8323/HALL_W -> /drv8323/HALL_V
- U10 pad 4: /stm32g431cb/SS_DRV -> /stm32g431cb/DRV_ENABLE
- U10 pad 41: /drv8323/HALL_V -> /drv8323/HALL_W
- U4 pad 10: /drv8323/SPI1_MOSI -> /drv8323/SPI2_MOSI
- U4 pad 11: /drv8323/SPI1_MISO -> /drv8323/SPI2_MISO
- U4 pad 9: /drv8323/SPI1_CLK -> /drv8323/SPI2_CLK
Routing:
- net GND: track 1047.2 -> 875.6 mm, vias 106 -> 113
- net +3.3V: track 89.1 -> 37.6 mm, vias 5 -> 9
- net /stm32g431cb/SS_DRV: track 49.8 -> 0.00 mm, vias 2 -> 0
- net /stm32g431cb/DRV_ENABLE: track 45.7 -> 0.00 mm, vias 2 -> 0
- net /stm32g431cb/FAULTB: track 30.8 -> 0.00 mm, vias 2 -> 0
- net /drv8323/SPI1_CLK: track 59.9 -> 29.5 mm, vias 3 -> 2
- net /drv8323/SPI1_MOSI: track 64.8 -> 35.5 mm, vias 3 -> 2
- net /stm32g431cb/ADC1_3: track 28.9 -> 0.00 mm, vias 2 -> 0
- net /drv8323/SPI1_MISO: track 66.8 -> 38.2 mm, vias 3 -> 2
- net /stm32g431cb/ADC1_2: track 26.8 -> 0.00 mm, vias 2 -> 0
- net /drv8323/INHB: track 71.8 -> 46.9 mm
- net /drv8323/INHA: track 76.4 -> 52.7 mm
- net /stm32g431cb/ADC1_1: track 23.7 -> 0.00 mm, vias 2 -> 0
- net /drv8323/INHC: track 61.4 -> 41.9 mm
- net /drv8323/SPI2_MISO: track 0.00 -> 19.0 mm, vias 0 -> 1
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- removed copper zone on In2.Cu, net GND
Other:
- board size 55 x 55 mm -> 50 x 50 mm

Commit message: chore: commit before starting to develop v1.2
Parts:
- moved R15 0.68 mm to (117.7, 105.1)
- moved C20 0.68 mm to (118.2, 107.1)
- moved C21 0.68 mm to (117.6, 109.2)
- moved Y1 0.68 mm to (116.6, 107.1)
- moved C10 0.61 mm to (101.0, 105.4)
Routing:
- net /stm32g431cb/FAULTB: track 0.00 -> 39.3 mm, vias 0 -> 2
- net /stm32g431cb/ADC1_3: track 0.00 -> 33.5 mm, vias 0 -> 2
- net /stm32g431cb/ADC1_2: track 0.00 -> 30.9 mm, vias 0 -> 2
- net /stm32g431cb/SS_DRV: track 0.00 -> 30.5 mm, vias 0 -> 2
- net /stm32g431cb/ADC1_1: track 0.00 -> 30.1 mm, vias 0 -> 2
- net /stm32g431cb/DRV_ENABLE: track 0.00 -> 29.0 mm, vias 0 -> 2
- net +3.3V: track 37.6 -> 44.9 mm, vias 9 -> 8
- net /drv8323/GHA: track 29.8 -> 34.7 mm
- net GND: track 875.6 -> 871.3 mm, vias 113 -> 105
- net /stm32g431cb/DRV_CAL: track 21.5 -> 24.2 mm
- net /stm32g431cb/OSC_OUT: track 9.00 -> 10.5 mm
- net /stm32g431cb/INLX: track 24.5 -> 25.7 mm
- net /stm32g431cb/NRST: track 58.4 -> 59.6 mm
- net /stm32g431cb/OSC_IN: track 4.90 -> 5.80 mm
- net +3.3VA: track 72.8 -> 73.6 mm
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- added copper zone on In2.Cu, net GND
