File: pcb/motor_driver/motor_driver.kicad_sch (KiCad schematic)
At the start: 19 parts

Commit message: update pcb
Parts:
- removed C? (x2): 2.2u, Capacitor_SMD:C_0402_1005Metric, symbol Device:C_Small
- removed C? (x6): 0.1u, Capacitor_SMD:C_0201_0603Metric, symbol Device:C_Small
- removed C? (x2): 15p, symbol Device:C_Small
- removed C?: 4.7u, Capacitor_SMD:C_0402_1005Metric, symbol Device:C_Small
- removed C?: 0.01u, Capacitor_SMD:C_0402_1005Metric, symbol Device:C_Small
- removed C?: 1u, Capacitor_SMD:C_0201_0603Metric, symbol Device:C_Small
- removed R?: 1k, symbol Device:R_Small
- removed R?: 330, symbol Device:R_Small
- removed R?: 10k, symbol Device:R_Small
- removed SW?: TVAF06-A020B-R, half_mouse_lib:TVAF06-A020B-R, symbol My_Device:SKRPACE
- removed U?: STM32G431CB, symbol bldc_lib:STM32G431CB
- removed Y?: 16MHz, symbol Device:Crystal_GND2_Small
- added J1: XT60PW-M, bldc_lib:XT60PWM, symbol bldc_lib:XT60PW-M
Connections:
- net GND: now also J1.1
- new net +BATT: J1.2
- no-connect marks 0 -> 2
Other:
- removed sheet COM
- removed sheet can
- removed sheet user_interface
- added sheet stm32g431cb (stm32g431cb.kicad_sch)
- sheet drv8323 ports: added FAULTB, HALL_U, HALL_V, HALL_W, SPI1_CLK, SPI1_MISO, SPI1_MOSI, SS_DRV, SS_ENC; removed SCLK, SDI, SDO, nFAULT, nSCS

Commit message: update pcb
Parts:
- J1: footprint bldc_lib:XT60PWM -> Connector_AMASS:AMASS_XT60-M_1x02_P7.20mm_Vertical
Changed lines of the file:
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@@
     (property "Reference" "J1" (id 0) (at 86.36 72.39 0))
     (property "Value" "XT60PW-M" (id 1) (at 86.36 74.93 0))
-    (property "Footprint" "bldc_lib:XT60PWM" (id 2) (at 76.2 80.01 0)
+    (property "Footprint" "Connector_AMASS:AMASS_XT60-M_1x02_P7.20mm_Vertical" (id 2) (at 76.2 80.01 0)
       (effects (font (size 1.27 1.27)) hide)
     )
@@
       (reference "C30") (unit 1) (value "0.1u") (footprint "Capacitor_SMD:C_0201_0603Metric")
     )
-    (path "/1bfc5921-cf85-4de6-a016-ca357e556864/c1c4533e-120d-4824-964a-a347c663c13e"
-      (reference "C31") (unit 1) (value "0.1u") (footprint "Capacitor_SMD:C_0201_0603Metric")
-    )
-    (path "/1bfc5921-cf85-4de6-a016-ca357e556864/5d6eb83b-ad05-4a82-ba02-33d920b6ce53"
-      (reference "C32") (unit 1) (value "0.1u") (footprint "Capacitor_SMD:C_0201_0603Metric")
-    )
     (path "/1bfc5921-cf85-4de6-a016-ca357e556864/b1529761-3313-4524-b7fd-63bd5b02efb6"
       (reference "C33") (unit 1) (value "0.1u") (footprint "Capacitor_SMD:C_0603_1608Metric_Pad1.08x0.95mm_HandSolder")
     )
     (path "/1bfc5921-cf85-4de6-a016-ca357e556864/8fb4f730-ee42-4237-9a8d-e3a3cee955eb"
-      (reference "C34") (unit 1) (value "0.01u") (footprint "Capacitor_SMD:C_0402_1005Metric")
-    )
-    (path "/1bfc5921-cf85-4de6-a016-ca357e556864/7a573b00-a11b-46eb-bfc9-add9107c6f47"
-      (reference "C35") (unit 1) (value "1u") (footprint "Capacitor_SMD:C_0201_0603Metric")
+      (reference "C34") (unit 1) (value "0.1u") (footprint "Capacitor_SMD:C_0402_1005Metric")
     )
     (path "/1bfc5921-cf85-4de6-a016-ca357e556864/7ba63036-3e3f-4395-bc39-ac84271a494f"
-      (reference "C36") (unit 1) (value "0.1u") (footprint "Capacitor_SMD:C_0603_1608Metric_Pad1.08x0.95mm_HandSolder")
+      (reference "C36") (unit 1) (value "0.1u") (footprint "Capacitor_SMD:C_0201_0603Metric")
     )
     (path "/99868341-3fcd-422d-afe6-e3750b4ef7c0/399c42df-e1bd-4dbb-84c7-161cbdbd03c4"
@@
     )
     (path "/fbfdd99d-8079-4968-88cb-ff84defd7944"
-      (reference "J1") (unit 1) (value "XT60PW-M") (footprint "bldc_lib:XT60PWM")
+      (reference "J1") (unit 1) (value "XT60PW-M") (footprint "Connector_AMASS:AMASS_XT60-M_1x02_P7.20mm_Vertical")
     )
     (path "/99868341-3fcd-422d-afe6-e3750b4ef7c0/dea1dc94-a988-4d20-b1f0-a54ceb254ec6"
@@
       (reference "Q1") (unit 1) (value "BSS138") (footprint "Package_TO_SOT_SMD:SOT-23")
     )
+    (path "/99868341-3fcd-422d-afe6-e3750b4ef7c0/c1d3f6fe-6174-4e55-ae26-b83d40fd6fd8"
+      (reference "Q2") (unit 1) (value "HP8K22TB") (footprint "bldc_lib:HP8K24TB")
+    )
+    (path "/99868341-3fcd-422d-afe6-e3750b4ef7c0/39c0be35-2c00-45ee-909c-14e12b3a55a5"
+      (reference "Q3") (unit 1) (value "HP8K22TB") (footprint "bldc_lib:HP8K24TB")
+    )
+    (path "/99868341-3fcd-422d-afe6-e3750b4ef7c0/8bc932f4-fa5d-4500-8309-6fb0c39b14c6"
+      (reference "Q4") (unit 1) (value "HP8K22TB") (footprint "bldc_lib:HP8K24TB")
+    )
     (path "/99868341-3fcd-422d-afe6-e3750b4ef7c0/b926b0e4-c3c8-4a72-b4ed-727b1ddbc7f9"
       (reference "R1") (unit 1) (value "1k") (footprint "Resistor_SMD:R_0402_1005Metric_Pad0.72x0.64mm_HandSolder")
@@
       (reference "U4") (unit 1) (value "a1333") (footprint "Package_SO:HTSSOP-14-1EP_4.4x5mm_P0.65mm_EP3.4x5mm_Mask3x3.1mm")
     )
-    (path "/99868341-3fcd-422d-afe6-e3750b4ef7c0/c1d3f6fe-6174-4e55-ae26-b83d40fd6fd8"
-      (reference "U5") (unit 1) (value "HP8K22TB") (footprint "bldc_lib:HP8K24TB")
-    )
-    (path "/99868341-3fcd-422d-afe6-e3750b4ef7c0/39c0be35-2c00-45ee-909c-14e12b3a55a5"
-      (reference "U6") (unit 1) (value "HP8K22TB") (footprint "bldc_lib:HP8K24TB")
-    )
-    (path "/99868341-3fcd-422d-afe6-e3750b4ef7c0/8bc932f4-fa5d-4500-8309-6fb0c39b14c6"
-      (reference "U7") (unit 1) (value "HP8K22TB") (footprint "bldc_lib:HP8K24TB")
-    )
     (path "/51484c10-a339-47e4-a28f-1fe6df54aaa5/9f440fdd-5449-4ac7-b342-8aa552208d75"

Commit message: feat: fix most bug
Parts:
- added H1, H2, H3, H4: MountingHole, MountingHole:MountingHole_3.2mm_M3_Pad_TopBottom, symbol Mechanical:MountingHole
Other:
- sheet drv8323 ports: added SPI2_CLK, SPI2_MISO, SPI2_MOSI; removed none
- sheet stm32g431cb ports: added SPI2_CLK, SPI2_MISO, SPI2_MOSI; removed none
Changed lines of the file:
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@@
+    (stroke (width 0) (type default) (color 0 0 0 0))
+  )
+  (wire (pts (xy 147.32 138.43) (xy 158.75 138.43))
     (stroke (width 0) (type default) (color 0 0 0 0))
   )
@@
     (stroke (width 0) (type default) (color 0 0 0 0))
   )
+  (wire (pts (xy 147.32 133.35) (xy 158.75 133.35))
+    (stroke (width 0) (type default) (color 0 0 0 0))
+  )
   (wire (pts (xy 147.32 127) (xy 158.75 127))
     (stroke (width 0) (type default) (color 0 0 0 0))
@@
     (stroke (width 0) (type default) (color 0 0 0 0))
   )
+  (wire (pts (xy 147.32 135.89) (xy 158.75 135.89))
+    (stroke (width 0) (type default) (color 0 0 0 0))
+  )
   (wire (pts (xy 147.32 109.22) (xy 158.75 109.22))
     (stroke (width 0) (type default) (color 0 0 0 0))
@@
   (wire (pts (xy 147.32 100.33) (xy 158.75 100.33))
     (stroke (width 0) (type default) (color 0 0 0 0))
+  )
+  (symbol (lib_id "Mechanical:MountingHole") (at 71.12 106.68 0) (unit 1)
+    (in_bom yes) (on_board yes) (fields_autoplaced)
+    (property "Reference" "H1" (id 0) (at 73.66 105.4099 0)
+      (effects (font (size 1.27 1.27)) (justify left))
+    )
+    (property "Value" "MountingHole" (id 1) (at 73.66 107.9499 0)
+      (effects (font (size 1.27 1.27)) (justify left))
+    )
+    (property "Footprint" "MountingHole:MountingHole_3.2mm_M3_Pad_TopBottom" (id 2) (at 71.12 106.68 0)
+      (effects (font (size 1.27 1.27)) hide)
+    )
+    (property "Datasheet" "~" (id 3) (at 71.12 106.68 0)
+      (effects (font (size 1.27 1.27)) hide)
+    )
+  )
+  (symbol (lib_id "Mechanical:MountingHole") (at 71.12 127 0) (unit 1)
+    (in_bom yes) (on_board yes) (fields_autoplaced)
+    (property "Reference" "H4" (id 0) (at 73.66 125.7299 0)
+      (effects (font (size 1.27 1.27)) (justify left))
+    )
+    (property "Value" "MountingHole" (id 1) (at 73.66 128.2699 0)
+      (effects (font (size 1.27 1.27)) (justify left))
+    )
+    (property "Footprint" "MountingHole:MountingHole_3.2mm_M3_Pad_TopBottom" (id 2) (at 71.12 127 0)
+      (effects (font (size 1.27 1.27)) hide)
+    )
+    (property "Datasheet" "~" (id 3) (at 71.12 127 0)
+      (effects (font (size 1.27 1.27)) hide)
+    )
   )
   (symbol (lib_id "power:+BATT") (at 68.58 73.66 0) (unit 1)
@@
     )
     (pin "1")
+  )
+  (symbol (lib_id "Mechanical:MountingHole") (at 71.12 120.65 0) (unit 1)
+    (in_bom yes) (on_board yes) (fields_autoplaced)
+    (property "Reference" "H3" (id 0) (at 73.66 119.3799 0)
+      (effects (font (size 1.27 1.27)) (justify left))
+    )
+    (property "Value" "MountingHole" (id 1) (at 73.66 121.9199 0)
+      (effects (font (size 1.27 1.27)) (justify left))
+    )
+    (property "Footprint" "MountingHole:MountingHole_3.2mm_M3_Pad_TopBottom" (id 2) (at 71.12 120.65 0)
+      (effects (font (size 1.27 1.27)) hide)
+    )
+    (property "Datasheet" "~" (id 3) (at 71.12 120.65 0)
+      (effects (font (size 1.27 1.27)) hide)
+    )
+  )
+  (symbol (lib_id "Mechanical:MountingHole") (at 71.12 113.03 0) (unit 1)
+    (in_bom yes) (on_board yes) (fields_autoplaced)
+    (property "Reference" "H2" (id 0) (at 73.66 111.7599 0)
+      (effects (font (size 1.27 1.27)) (justify left))
+    )
+    (property "Value" "MountingHole" (id 1) (at 73.66 114.2999 0)
+      (effects (font (size 1.27 1.27)) (justify left))
+    )
+    (property "Footprint" "MountingHole:MountingHole_3.2mm_M3_Pad_TopBottom" (id 2) (at 71.12 113.03 0)
+      (effects (font (size 1.27 1.27)) hide)
+    )
+    (property "Datasheet" "~" (id 3) (at 71.12 113.03 0)
+      (effects (font (size 1.27 1.27)) hide)
+    )
   )
   (symbol (lib_id "power:GND") (at 72.39 90.17 0) (unit 1)
@@
     (pin "4")
   )
-  (sheet (at 113.03 69.85) (size 34.29 63.5) (fields_autoplaced)
+  (sheet (at 113.03 69.85) (size 34.29 71.12) (fields_autoplaced)
     (stroke (width 0.1524) (type solid) (color 0 0 0 0))
     (fill (color 0 0 0 0.0000))
@@
       (effects (font (size 1.27 1.27)) (justify left bottom))
     )
-    (property "Sheet file" "stm32g431cb.kicad_sch" (id 1) (at 113.03 133.9346 0)
+    (property "Sheet file" "stm32g431cb.kicad_sch" (id 1) (at 113.03 141.5546 0)
       (effects (font (size 1.27 1.27)) (justify left top))
     )
@@
     )
     (pin "SOA" input (at 147.32 91.44 0)
+      (effects (font (size 1.27 1.27)) (justify right))
+    )
+    (pin "SPI2_MOSI" input (at 147.32 135.89 0)
+      (effects (font (size 1.27 1.27)) (justify right))
+    )
+    (pin "SPI2_CLK" input (at 147.32 133.35 0)
+      (effects (font (size 1.27 1.27)) (justify right))
+    )
+    (pin "SPI2_MISO" input (at 147.32 138.43 0)
       (effects (font (size 1.27 1.27)) (justify right))
     )
@@
     )
   )
-  (sheet (at 158.75 69.85) (size 29.21 63.5) (fields_autoplaced)
+  (sheet (at 158.75 69.85) (size 29.21 71.12) (fields_autoplaced)
     (stroke (width 0.1524) (type solid) (color 0 0 0 0))
     (fill (color 0 0 0 0.0000))
@@
       (effects (font (size 1.27 1.27)) (justify left bottom))
     )
-    (property "Sheet file" "drv8323.kicad_sch" (id 1) (at 158.75 133.9346 0)
+    (property "Sheet file" "drv8323.kicad_sch" (id 1) (at 158.75 141.5546 0)
       (effects (font (size 1.27 1.27)) (justify left top))
     )
@@
     )
     (pin "INLB" input (at 158.75 85.09 180)
+      (effects (font (size 1.27 1.27)) (justify left))
+    )
+    (pin "SPI2_MOSI" input (at 158.75 135.89 180)
+      (effects (font (size 1.27 1.27)) (justify left))
+    )
+    (pin "SPI2_CLK" input (at 158.75 133.35 180)
+      (effects (font (size 1.27 1.27)) (justify left))
+    )
+    (pin "SPI2_MISO" input (at 158.75 138.43 180)
       (effects (font (size 1.27 1.27)) (justify left))
     )
@@
       (reference "#PWR083") (unit 1) (value "GND") (footprint "")
     )
-    (path "/1bfc5921-cf85-4de6-a016-ca357e556864/f5fe5de5-062c-4251-a450-c80b3c186252"
-      (reference "#PWR084") (unit 1) (value "GND") (footprint "")
-    )
-    (path "/1bfc5921-cf85-4de6-a016-ca357e556864/f2a62155-bb78-4818-90dc-ffe84b6efa9f"
-      (reference "#PWR085") (unit 1) (value "+3.3V") (footprint "")
-    )
     (path "/1bfc5921-cf85-4de6-a016-ca357e556864/a7c2bc4a-edee-41fc-b59b-a2b20db112a7"
       (reference "#PWR086") (unit 1) (value "+5V") (footprint "")
@@
     )
     (path "/99868341-3fcd-422d-afe6-e3750b4ef7c0/99ec7d60-c371-43f0-98e0-90688dc89eda"
-      (reference "#PWR?") (unit 1) (value "GND") (footprint "")
+      (reference "#PWR0101") (unit 1) (value "GND") (footprint "")
     )
     (path "/99868341-3fcd-422d-afe6-e3750b4ef7c0/9985f713-fca9-4262-a1f9-5f54a82a0e32"
@@
       (reference "D10") (unit 1) (value "LED6") (footprint "LED_SMD:LED_0402_1005Metric")
     )
+    (path "/157e2423-acea-4de2-831f-7936c63c850b"
+      (reference "H1") (unit 1) (value "MountingHole") (footprint "MountingHole:MountingHole_3.2mm_M3_Pad_TopBottom")
+    )
+    (path "/b7e7c0eb-4ecf-4a05-903e-7a0636efb463"
+      (reference "H2") (unit 1) (value "MountingHole") (footprint "MountingHole:MountingHole_3.2mm_M3_Pad_TopBottom")
+    )
+    (path "/a2f18580-cb62-4f19-93cd-a733956954e5"
+      (reference "H3") (unit 1) (value "MountingHole") (footprint "MountingHole:MountingHole_3.2mm_M3_Pad_TopBottom")
+    )
+    (path "/558a832f-ac1d-4c17-a487-d12b92fd2d8c"
+      (reference "H4") (unit 1) (value "MountingHole") (footprint "MountingHole:MountingHole_3.2mm_M3_Pad_TopBottom")
+    )
     (path "/fbfdd99d-8079-4968-88cb-ff84defd7944"
       (reference "J1") (unit 1) (value "XT60PW-M") (footprint "Connector_AMASS:AMASS_XT60-M_1x02_P7.20mm_Vertical")
@@
       (reference "J3") (unit 1) (value "Conn_ARM_JTAG_SWD_10") (footprint "Connector_PinHeader_1.27mm:PinHeader_2x05_P1.27mm_Vertical")
     )
-    (path "/1bfc5921-cf85-4de6-a016-ca357e556864/7aef4efb-61aa-42e5-9d72-13c39081d1b7"
-      (reference "J4") (unit 1) (value "UART1 SH") (footprint "Connector_PinHeader_2.54mm:PinHeader_1x04_P2.54mm_Vertical")
-    )
     (path "/1bfc5921-cf85-4de6-a016-ca357e556864/cddc824b-d9d8-43da-abbe-7929fd2a031f"
