File: pcb/motor_driver/power.kicad_sch (KiCad schematic)
At the start: 6 parts

Commit message: update pcb
Parts:
- removed C? (x2): 10u, symbol Device:C_Small
- removed D? (x2): SS2040, Diode_SMD:D_MELF, symbol Diode:1N5712UR
- removed J?: Conn_01x02_Female, symbol Connector:Conn_01x02_Female
- removed U?: R-78E5.0-0.5, symbol bldc_lib:R-78E5.0-0.5
- added C14, C17: 0.01u, Capacitor_SMD:C_0603_1608Metric_Pad1.08x0.95mm_HandSolder, symbol Device:C_Small
- added C15, C16, C18, C19: 1u, Capacitor_SMD:C_0603_1608Metric_Pad1.08x0.95mm_HandSolder, symbol Device:C_Small
- added D4: LED, LED_SMD:LED_0603_1608Metric_Pad1.05x0.95mm_HandSolder, symbol Device:LED
- added R13: 1k, Resistor_SMD:R_0402_1005Metric_Pad0.72x0.64mm_HandSolder, symbol Device:R_Small
- added U8: ADP151AUJZ-3.3-R7, Package_TO_SOT_SMD:SOT-23-5_HandSoldering, symbol bldc_lib:ADP151AUJZ-3.3-R7
- added U9: NJM12877F33-TE1, Package_TO_SOT_SMD:SOT-23-5_HandSoldering, symbol bldc_lib:NJM12877F33-TE1
Connections:
- net +5V: now also C14.1, C15.1, C16.1, U8.1 (VIN), U8.3 (EN), U9.1 (VIN), U9.3 (CONTROL)
- net GND: now also C14.2, C15.2, C16.2, C17.2, C18.2, C19.2, R13.2, U8.2 (GND), U9.2 (GND)
- new net: C17.1, U9.4 (Cs)
- new net: D4.1 (K), R13.1
- new net +3.3V: C18.1, D4.2 (A), U9.5 (VOUT)
- new net +3.3VA: C19.1, U8.5 (VOUT)
