File: pcb/main/can_connector.kicad_sch (KiCad schematic)
At the start: 5 parts

Commit message: chore: add circuit git changes
Parts:
- removed D?: LED5, LED_SMD:LED_0402_1005Metric, symbol Device:LED
- removed D?: LED6, LED_SMD:LED_0402_1005Metric, symbol Device:LED
- removed J?: Conn_01x04_Female, symbol Connector:Conn_01x04_Female
- removed R? (x2): 1k, Resistor_SMD:R_0201_0603Metric, symbol Device:R_Small
- added J?: Conn, bldc_lib:21322604YY, symbol Connector_Generic:Conn_01x06
Connections:
- net +5V: now also J?.1 (Pin_1)
- net CAN_H: now also J?.3 (Pin_3)
- net CAN_L: now also J?.2 (Pin_2)
- net GND: now also J?.4 (Pin_4), J?.5 (Pin_5), J?.6 (Pin_6)
Changed lines of the file:
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@@
 (kicad_sch (version 20211123) (generator eeschema)
   (paper "A4")
-  (wire (pts (xy 181.61 71.12) (xy 181.61 77.47))
+  (junction (at 134.62 92.71) (diameter 0) (color 0 0 0 0)
+  )
+  (junction (at 134.62 90.17) (diameter 0) (color 0 0 0 0)
+  )
+  (wire (pts (xy 134.62 92.71) (xy 139.7 92.71))
     (stroke (width 0) (type default) (color 0 0 0 0))
   )
-  (wire (pts (xy 191.77 71.12) (xy 191.77 77.47))
+  (wire (pts (xy 134.62 92.71) (xy 134.62 96.52))
     (stroke (width 0) (type default) (color 0 0 0 0))
   )
-  (wire (pts (xy 181.61 90.17) (xy 181.61 93.98))
+  (wire (pts (xy 134.62 80.01) (xy 139.7 80.01))
     (stroke (width 0) (type default) (color 0 0 0 0))
   )
-  (wire (pts (xy 191.77 90.17) (xy 191.77 93.98))
+  (wire (pts (xy 134.62 80.01) (xy 134.62 78.74))
     (stroke (width 0) (type default) (color 0 0 0 0))
   )
-  (wire (pts (xy 127 87.63) (xy 127 91.44))
+  (wire (pts (xy 134.62 87.63) (xy 139.7 87.63))
     (stroke (width 0) (type default) (color 0 0 0 0))
   )
-  (wire (pts (xy 130.81 87.63) (xy 127 87.63))
+  (wire (pts (xy 134.62 90.17) (xy 139.7 90.17))
     (stroke (width 0) (type default) (color 0 0 0 0))
   )
-  (wire (pts (xy 127 80.01) (xy 127 76.2))
+  (wire (pts (xy 134.62 90.17) (xy 134.62 92.71))
     (stroke (width 0) (type default) (color 0 0 0 0))
   )
-  (wire (pts (xy 130.81 80.01) (xy 127 80.01))
+  (wire (pts (xy 134.62 87.63) (xy 134.62 90.17))
     (stroke (width 0) (type default) (color 0 0 0 0))
   )
-  (hierarchical_label "LED_RX" (shape input) (at 191.77 71.12 90)
-    (effects (font (size 1.27 1.27)) (justify left))
-  )
-  (hierarchical_label "LED_TX" (shape input) (at 181.61 71.12 90)
-    (effects (font (size 1.27 1.27)) (justify left))
-  )
-  (hierarchical_label "CAN_H" (shape input) (at 130.81 82.55 180)
+  (hierarchical_label "CAN_L" (shape input) (at 139.7 82.55 180)
     (effects (font (size 1.27 1.27)) (justify right))
   )
-  (hierarchical_label "CAN_L" (shape input) (at 130.81 85.09 180)
+  (hierarchical_label "CAN_H" (shape input) (at 139.7 85.09 180)
     (effects (font (size 1.27 1.27)) (justify right))
   )
-  (symbol (lib_id "Connector:Conn_01x04_Female") (at 135.89 82.55 0) (unit 1)
+  (symbol (lib_id "power:+5V") (at 134.62 78.74 0) (unit 1)
     (in_bom yes) (on_board yes) (fields_autoplaced)
-    (property "Reference" "J?" (id 0) (at 137.16 82.5499 0)
+    (property "Reference" "#PWR?" (id 0) (at 134.62 82.55 0)
+      (effects (font (size 1.27 1.27)) hide)
+    )
+    (property "Value" "+5V" (id 1) (at 134.62 73.66 0))
+    (property "Footprint" "" (id 2) (at 134.62 78.74 0)
+      (effects (font (size 1.27 1.27)) hide)
+    )
+    (property "Datasheet" "" (id 3) (at 134.62 78.74 0)
+      (effects (font (size 1.27 1.27)) hide)
+    )
+    (pin "1")
+  )
+  (symbol (lib_id "power:GND") (at 134.62 96.52 0) (unit 1)
+    (in_bom yes) (on_board yes) (fields_autoplaced)
+    (property "Reference" "#PWR?" (id 0) (at 134.62 102.87 0)
+      (effects (font (size 1.27 1.27)) hide)
+    )
+    (property "Value" "GND" (id 1) (at 134.62 101.6 0))
+    (property "Footprint" "" (id 2) (at 134.62 96.52 0)
+      (effects (font (size 1.27 1.27)) hide)
+    )
+    (property "Datasheet" "" (id 3) (at 134.62 96.52 0)
+      (effects (font (size 1.27 1.27)) hide)
+    )
+    (pin "1")
+  )
+  (symbol (lib_id "Connector_Generic:Conn_01x06") (at 144.78 85.09 0) (unit 1)
+    (in_bom yes) (on_board yes)
+    (property "Reference" "J?" (id 0) (at 146.812 85.2932 0)
       (effects (font (size 1.27 1.27)) (justify left))
     )
-    (property "Value" "Conn_01x04_Female" (id 1) (at 137.16 85.0899 0)
+    (property "Value" "Conn" (id 1) (at 146.812 87.6046 0)
       (effects (font (size 1.27 1.27)) (justify left))
     )
-    (property "Footprint" "" (id 2) (at 135.89 82.55 0)
+    (property "Footprint" "bldc_lib:21322604YY" (id 2) (at 144.78 85.09 0)
       (effects (font (size 1.27 1.27)) hide)
     )
-    (property "Datasheet" "~" (id 3) (at 135.89 82.55 0)
+    (property "Datasheet" "~" (id 3) (at 144.78 85.09 0)
       (effects (font (size 1.27 1.27)) hide)
     )
@@
     (pin "3")
     (pin "4")
-  )
-  (symbol (lib_id "power:+5V") (at 127 76.2 0) (unit 1)
-    (in_bom yes) (on_board yes) (fields_autoplaced)
-    (property "Reference" "#PWR?" (id 0) (at 127 80.01 0)
-      (effects (font (size 1.27 1.27)) hide)
-    )
-    (property "Value" "+5V" (id 1) (at 127 71.12 0))
-    (property "Footprint" "" (id 2) (at 127 76.2 0)
-      (effects (font (size 1.27 1.27)) hide)
-    )
-    (property "Datasheet" "" (id 3) (at 127 76.2 0)
-      (effects (font (size 1.27 1.27)) hide)
-    )
-    (pin "1")
-  )
-  (symbol (lib_id "power:GND") (at 127 91.44 0) (unit 1)
-    (in_bom yes) (on_board yes) (fields_autoplaced)
-    (property "Reference" "#PWR?" (id 0) (at 127 97.79 0)
-      (effects (font (size 1.27 1.27)) hide)
-    )
-    (property "Value" "GND" (id 1) (at 127 96.52 0))
-    (property "Footprint" "" (id 2) (at 127 91.44 0)
-      (effects (font (size 1.27 1.27)) hide)
-    )
-    (property "Datasheet" "" (id 3) (at 127 91.44 0)
-      (effects (font (size 1.27 1.27)) hide)
-    )
-    (pin "1")
-  )
-  (symbol (lib_id "power:GND") (at 181.61 93.98 0) (unit 1)
-    (in_bom yes) (on_board yes) (fields_autoplaced)
-    (property "Reference" "#PWR?" (id 0) (at 181.61 100.33 0)
-      (effects (font (size 1.27 1.27)) hide)
-    )
-    (property "Value" "GND" (id 1) (at 181.61 99.06 0))
-    (property "Footprint" "" (id 2) (at 181.61 93.98 0)
-      (effects (font (size 1.27 1.27)) hide)
-    )
-    (property "Datasheet" "" (id 3) (at 181.61 93.98 0)
-      (effects (font (size 1.27 1.27)) hide)
-    )
-    (pin "1")
-  )
-  (symbol (lib_id "Device:R_Small") (at 191.77 80.01 0) (unit 1)
-    (in_bom yes) (on_board yes) (fields_autoplaced)
-    (property "Reference" "R?" (id 0) (at 194.31 78.7399 0)
-      (effects (font (size 1.27 1.27)) (justify left))
-    )
-    (property "Value" "1k" (id 1) (at 194.31 81.2799 0)
-      (effects (font (size 1.27 1.27)) (justify left))
-    )
-    (property "Footprint" "Resistor_SMD:R_0201_0603Metric" (id 2) (at 191.77 80.01 0)
-      (effects (font (size 1.27 1.27)) hide)
-    )
-    (property "Datasheet" "~" (id 3) (at 191.77 80.01 0)
-      (effects (font (size 1.27 1.27)) hide)
-    )
-    (pin "1")
-    (pin "2")
-  )
-  (symbol (lib_id "Device:LED") (at 181.61 86.36 90) (unit 1)
-    (in_bom yes) (on_board yes) (fields_autoplaced)
-    (property "Reference" "D?" (id 0) (at 185.42 86.6774 90)
-      (effects (font (size 1.27 1.27)) (justify right))
-    )
-    (property "Value" "LED5" (id 1) (at 185.42 89.2174 90)
-      (effects (font (size 1.27 1.27)) (justify right))
-    )
-    (property "Footprint" "LED_SMD:LED_0402_1005Metric" (id 2) (at 181.61 86.36 0)
-      (effects (font (size 1.27 1.27)) hide)
-    )
-    (property "Datasheet" "~" (id 3) (at 181.61 86.36 0)
-      (effects (font (size 1.27 1.27)) hide)
-    )
-    (pin "1")
-    (pin "2")
-  )
-  (symbol (lib_id "Device:LED") (at 191.77 86.36 90) (unit 1)
-    (in_bom yes) (on_board yes) (fields_autoplaced)
-    (property "Reference" "D?" (id 0) (at 195.58 86.6774 90)
-      (effects (font (size 1.27 1.27)) (justify right))
-    )
-    (property "Value" "LED6" (id 1) (at 195.58 89.2174 90)
-      (effects (font (size 1.27 1.27)) (justify right))
-    )
-    (property "Footprint" "LED_SMD:LED_0402_1005Metric" (id 2) (at 191.77 86.36 0)
-      (effects (font (size 1.27 1.27)) hide)
-    )
-    (property "Datasheet" "~" (id 3) (at 191.77 86.36 0)
-      (effects (font (size 1.27 1.27)) hide)
-    )
-    (pin "1")
-    (pin "2")
-  )
-  (symbol (lib_id "Device:R_Small") (at 181.61 80.01 0) (unit 1)
-    (in_bom yes) (on_board yes) (fields_autoplaced)
-    (property "Reference" "R?" (id 0) (at 184.15 78.7399 0)
-      (effects (font (size 1.27 1.27)) (justify left))
-    )
-    (property "Value" "1k" (id 1) (at 184.15 81.2799 0)
-      (effects (font (size 1.27 1.27)) (justify left))
-    )
-    (property "Footprint" "Resistor_SMD:R_0201_0603Metric" (id 2) (at 181.61 80.01 0)
-      (effects (font (size 1.27 1.27)) hide)
-    )
-    (property "Datasheet" "~" (id 3) (at 181.61 80.01 0)
-      (effects (font (size 1.27 1.27)) hide)
-    )
-    (pin "1")
-    (pin "2")
-  )
-  (symbol (lib_id "power:GND") (at 191.77 93.98 0) (unit 1)
-    (in_bom yes) (on_board yes) (fields_autoplaced)
-    (property "Reference" "#PWR?" (id 0) (at 191.77 100.33 0)
-      (effects (font (size 1.27 1.27)) hide)
-    )
-    (property "Value" "GND" (id 1) (at 191.77 99.06 0))
-    (property "Footprint" "" (id 2) (at 191.77 93.98 0)
-      (effects (font (size 1.27 1.27)) hide)
-    )
-    (property "Datasheet" "" (id 3) (at 191.77 93.98 0)
-      (effects (font (size 1.27 1.27)) hide)
-    )
-    (pin "1")
+    (pin "5")
+    (pin "6")
   )
 )
