File: pcb/main/imu_connector.kicad_sch (KiCad schematic)
At the start: 1 part

Commit message: chore: add circuit git changes
Parts:
- J2: renamed from J?; footprint (none) -> Connector_JST:JST_ZE_SM06B-ZESS-TB_1x06-1MP_P1.50mm_Horizontal
Changed lines of the file:
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@@
   (symbol (lib_id "power:+3.3V") (at 118.11 73.66 0) (unit 1)
     (in_bom yes) (on_board yes)
-    (property "Reference" "#PWR?" (id 0) (at 118.11 77.47 0)
+    (property "Reference" "#PWR03" (id 0) (at 118.11 77.47 0)
       (effects (font (size 1.27 1.27)) hide)
     )
@@
   (symbol (lib_id "power:GND") (at 118.11 93.98 0) (mirror y) (unit 1)
     (in_bom yes) (on_board yes)
-    (property "Reference" "#PWR?" (id 0) (at 118.11 100.33 0)
+    (property "Reference" "#PWR04" (id 0) (at 118.11 100.33 0)
       (effects (font (size 1.27 1.27)) hide)
     )
@@
   (symbol (lib_id "Connector:Conn_01x06_Female") (at 128.27 81.28 0) (unit 1)
     (in_bom yes) (on_board yes) (fields_autoplaced)
-    (property "Reference" "J?" (id 0) (at 129.54 81.2799 0)
+    (property "Reference" "J2" (id 0) (at 129.54 81.2799 0)
       (effects (font (size 1.27 1.27)) (justify left))
     )
@@
       (effects (font (size 1.27 1.27)) (justify left))
     )
-    (property "Footprint" "" (id 2) (at 128.27 81.28 0)
+    (property "Footprint" "Connector_JST:JST_ZE_SM06B-ZESS-TB_1x06-1MP_P1.50mm_Horizontal" (id 2) (at 128.27 81.28 0)
       (effects (font (size 1.27 1.27)) hide)
     )

Commit message: feat: finish main board v2
Parts:
- renumbered J2 to J7
