File: pcb/main/power.kicad_sch (KiCad schematic)
At the start: 11 parts, among them U1 NJM12877F33-TE1, U4 LXDC55FAAA-203

Commit message: feat: finish main board v2
Parts:
- removed C1: 0.01u, Capacitor_SMD:C_0603_1608Metric_Pad1.08x0.95mm_HandSolder, symbol Device:C_Small
- removed C2: 1u, Capacitor_SMD:C_0603_1608Metric_Pad1.08x0.95mm_HandSolder, symbol Device:C_Small
- removed U1: NJM12877F33-TE1, Package_TO_SOT_SMD:SOT-23-5_HandSoldering, symbol bldc_lib:NJM12877F33-TE1
- added D1: LED, LED_SMD:LED_0603_1608Metric, symbol Device:LED
- added R2: 1k, Resistor_SMD:R_0603_1608Metric_Pad0.98x0.95mm_HandSolder, symbol Device:R_Small
- added R25: 12k, Resistor_SMD:R_0603_1608Metric, symbol Device:R_Small
- added R26: 33k, Resistor_SMD:R_0603_1608Metric, symbol Device:R_Small
- added U2: LT1963AES3-3.3, Package_TO_SOT_SMD:SOT-223, symbol My_Device:LT1963AES3-3.3
- C2: renamed from C18; footprint Capacitor_SMD:C_0603_1608Metric_Pad1.08x0.95mm_HandSolder -> Capacitor_SMD:C_0805_2012Metric_Pad1.18x1.45mm_HandSolder
- C3: value 0.01u -> 10u; footprint Capacitor_SMD:C_0603_1608Metric_Pad1.08x0.95mm_HandSolder -> Capacitor_SMD:C_0805_2012Metric_Pad1.18x1.45mm_HandSolder
- C4: value 1u -> 10u; footprint Capacitor_SMD:C_0603_1608Metric_Pad1.08x0.95mm_HandSolder -> Capacitor_SMD:C_0805_2012Metric_Pad1.18x1.45mm_HandSolder
- C5: renamed from C19; footprint Capacitor_SMD:C_0603_1608Metric_Pad1.08x0.95mm_HandSolder -> Capacitor_SMD:C_0805_2012Metric_Pad1.18x1.45mm_HandSolder
- D2: renamed from D1; footprint LED_SMD:LED_0402_1005Metric -> LED_SMD:LED_0603_1608Metric
- R1: renamed from R22; footprint Resistor_SMD:R_0603_1608Metric_Pad0.98x0.95mm_HandSolder -> Resistor_SMD:R_0805_2012Metric
- renumbered R1 to R3, U4 to U1
Connections:
- net +3.3V: now also U2.3 (OUT)
- net +5V: now also C3.1, D1.2 (A), U2.1 (IN)
- net +BATT: now also R25.1
- net GND: now also R2.2, R26.2, U2.2 (GND), U2.4 (GND)
- new net: D1.1 (K), R2.1
- new net ADC_BATTERY: R25.2, R26.1
Other:
- moved on the sheet: D2, R3
