File: pcb/main/main.kicad_pcb (KiCad board)
At the start: 2 copper layers, 91 x 94.8 mm, 71 parts, among them J1 XT60PW-M, J10 Conn, J11 Conn_ARM_JTAG_SWD_10, J12 UART1 SH, J13 Micro_SD_Card, J14 PH 2.0, J2 Conn_01x06_Female, J3 Conn_01x06_Female, J4 Conn_01x06_Female, J5 Conn_01x06_Female, J6 Conn_01x06_Female, J7 Conn_01x06_Female, J8 Conn, J9 Conn, Q1 BSS138, SW1 RESET, SW2 USER, U1 NJM12877F33-TE1, U2 STM32F405RGTx, U3 MCP2562-E-SN, U4 LXDC55FAAA-203, Y1 XRCGB16M000FXN02R0

Commit message: perf: update LCD and microSD
Parts:
- J1: footprint Connector_AMASS:AMASS_XT30U-F_1x02_P5.0mm_Vertical -> Connector_AMASS:AMASS_XT60-F_1x02_P7.20mm_Vertical
- renumbered C17 to C1, C9 to C10, C10 to C11, C11 to C12, C12 to C13, C13 to C14, C14 to C15, C15 to C16, C5 to C17, C8 to C18, C16 to C19, C18 to C2, C1 to C3, C2 to C4, C19 to C5, C3 to C6, C4 to C7, C6 to C8, C7 to C9, J14 to J10, J13 to J9, R22 to R1, R5 to R10, R6 to R11, R7 to R12, R3 to R13, R8 to R14, R9 to R15, R10 to R16, R11 to R17, R12 to R18, R13 to R19, R1 to R2, R14 to R20, R15 to R21, R16 to R22, R2 to R3, R17 to R4, R18 to R5, R19 to R6, R20 to R7, R21 to R8, R4 to R9, U4 to U1, U1 to U2, U2 to U3, U3 to U4
Connections:
- C17 pad 1: Net-(C5-Pad1) -> (no net)
- C6 pad 1: Net-(C3-Pad1) -> (no net)
- C8 pad 1: Net-(C6-Pad1) -> (no net)
- C9 pad 1: Net-(C7-Pad1) -> (no net)
- J11 pad 6: unconnected-(J11-Pad6) -> (no net)
- J11 pad 7: unconnected-(J11-Pad7) -> (no net)
- J11 pad 8: unconnected-(J11-Pad8) -> (no net)
- Q1 pad 3: Net-(Q1-Pad3) -> (no net)
- R1 pad 1: Net-(R22-Pad1) -> (no net)
- R13 pad 2: Net-(C5-Pad1) -> Net-(C17-Pad1)
- R17 pad 2: Net-(R11-Pad2) (its old number) -> (no net)
- R3 pad 1: Net-(R2-Pad1) -> (no net)
- SP1 pad 2: Net-(Q1-Pad3) -> Net-(Q1-D)
- SW2 pad 1: Net-(R11-Pad2) (its old number) -> Net-(R17-Pad2)
- U1 pad 10: unconnected-(U4-Pad10) -> (no net)
- U1 pad 11: Net-(R22-Pad1) -> Net-(U1-FB)
- U1 pad 2: unconnected-(U4-Pad2) -> (no net)
- U2 pad 4: Net-(C3-Pad1) -> Net-(U2-Cs)
- U3 pad 20: unconnected-(U2-Pad20) -> (no net)
- U3 pad 24: unconnected-(U2-Pad24) -> (no net)
- U3 pad 29: unconnected-(U2-Pad29) -> (no net)
- U3 pad 3: unconnected-(U2-Pad3) -> (no net)
- U3 pad 31: Net-(C6-Pad1) -> Net-(U3-VCAP_1)
- U3 pad 33: unconnected-(U2-Pad33) -> (no net)
- U3 pad 36: unconnected-(U2-Pad36) -> (no net)
- U3 pad 37: unconnected-(U2-Pad37) -> (no net)
- U3 pad 4: unconnected-(U2-Pad4) -> (no net)
- U3 pad 47: Net-(C7-Pad1) -> Net-(U3-VCAP_2)
- U3 pad 50: unconnected-(U2-Pad50) -> (no net)
- U3 pad 60: Net-(R2-Pad1) -> Net-(U3-BOOT0)
- U3 pad 61: unconnected-(U2-Pad61) -> (no net)
- U3 pad 62: unconnected-(U2-Pad62) -> (no net)
- U3 pad 8: unconnected-(U2-Pad8) -> (no net)
- U3 pad 9: unconnected-(U2-Pad9) -> (no net)
- Y1 pad 1: Net-(C5-Pad1) -> Net-(C17-Pad1)
Routing:
- net Net-(U3-VCAP_1): track 0.00 -> 6.17 mm
- net Net-(C6-Pad1): track 6.17 -> 0.00 mm
- net Net-(U3-BOOT0): track 0.00 -> 5.34 mm
- net Net-(R2-Pad1): track 5.34 -> 0.00 mm
- net Net-(Q1-Pad3): track 4.44 -> 0.00 mm
- net Net-(Q1-D): track 0.00 -> 4.44 mm
- net Net-(C5-Pad1): track 3.38 -> 0.00 mm
- net Net-(C17-Pad1): track 0.00 -> 3.38 mm
- net Net-(U2-Cs): track 0.00 -> 3.17 mm
- net Net-(C3-Pad1): track 3.17 -> 0.00 mm
- net Net-(U3-VCAP_2): track 0.00 -> 2.46 mm
- net Net-(C7-Pad1): track 2.46 -> 0.00 mm
- net Net-(U1-FB): track 0.00 -> 2.38 mm
- net Net-(R22-Pad1): track 2.38 -> 0.00 mm
- net Net-(R17-Pad2): track 0.00 -> 2.22 mm
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