File: pcb/main/stm32f405rg.kicad_sch (KiCad schematic)
At the start: 49 parts, among them J11 Conn_ARM_JTAG_SWD_10, J12 UART1 SH, J13 Micro_SD_Card, J14 PH 2.0, Q1 BSS138, SW1 RESET, SW2 USER, U2 STM32F405RGTx, U3 MCP2562-E-SN, Y1 XRCGB16M000FXN02R0

Commit message: perf: update LCD and microSD
Parts:
- renumbered C9 to C10, C10 to C11, C11 to C12, C12 to C13, C13 to C14, C14 to C15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
