File: pcb/motor_driver/v1.2/drv8323.kicad_sch (KiCad schematic)
At the start: 27 parts, among them J2 1-84953-1, Q2 HP8K22TB, Q3 HP8K22TB, Q4 HP8K22TB, U3 DRV8323S, U4 a1333

Commit message: perf: fix pcb for v1.2
Parts:
- U1: renamed from U3; footprint Package_DFN_QFN:QFN-40-1EP_6x6mm_P0.5mm_EP4.6x4.6mm_ThermalVias -> Package_DFN_QFN:QFN-40-1EP_6x6mm_P0.5mm_EP4.6x4.6mm
- renumbered C11 to C10, C12 to C11, C13 to C12, C7 to C5, C10 to C7, J2 to J3, Q2 to Q1, Q3 to Q2, Q4 to Q3, R4 to R1, R5 to R2, R6 to R3, R7 to R4, R8 to R5, R9 to R6, R10 to R7, R11 to R8, R12 to R9, U4 to U2
Other:
- moved on the sheet: C7, C9

Commit message: perf: update motor driver pdb
Parts:
- C8: footprint Capacitor_SMD:CP_Elec_8x10.5 -> Capacitor_SMD:CP_Elec_6.3x3.9
Connections:
- net SOA: now also U1.21 (SOC); no longer U1.23 (SOA)
- net SOC: now also U1.23 (SOA); no longer U1.21 (SOC)
Changed lines of the file:
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@@
 		)
 	)
-	(hierarchical_label "SOC"
+	(hierarchical_label "SOA"
 		(shape output)
 		(at 118.11 71.12 0)
@@
 		)
 	)
-	(hierarchical_label "SOA"
+	(hierarchical_label "SOC"
 		(shape output)
 		(at 118.11 66.04 0)
@@
 			)
 		)
-		(property "Footprint" "Capacitor_SMD:CP_Elec_8x10.5"
+		(property "Footprint" "Capacitor_SMD:CP_Elec_6.3x3.9"
 			(at 191.77 149.86 0)
 			(effects

Commit message: feat: add additional CAN connetctor
Parts:
- renumbered J3 to J2
Changed lines of the file:
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@@
 		(dnp no)
 		(fields_autoplaced yes)
-		(property "Reference" "J3"
+		(property "Reference" "J2"
 			(at 104.14 104.14 0)
 			(effects
@@
 			(project "motor_driver"
 				(path "/1ef6600e-ea1d-4a9a-8ae5-1c3f7136836c/99868341-3fcd-422d-afe6-e3750b4ef7c0"
-					(reference "J3")
+					(reference "J2")
 					(unit 1)
 				)
