File: pcb/motor_driver/v1.2/power.kicad_sch (KiCad schematic)
At the start: 10 parts, among them U8 ADP151AUJZ-3.3-R7, U9 NJM12877F33-TE1

Commit message: perf: fix pcb for v1.2
Parts:
- D1: renamed from D4; footprint LED_SMD:LED_0603_1608Metric_Pad1.05x0.95mm_HandSolder -> LED_SMD:LED_0603_1608Metric
- R10: renamed from R13; footprint Resistor_SMD:R_0402_1005Metric_Pad0.72x0.64mm_HandSolder -> Resistor_SMD:R_0603_1608Metric_Pad0.98x0.95mm_HandSolder
- renumbered C14 to C13, C15 to C14, C16 to C15, C17 to C16, C18 to C17, C19 to C18, U8 to U3, U9 to U4
Changed lines of the file:
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@@
 		(dnp no)
 		(fields_autoplaced yes)
-		(property "Reference" "#PWR043"
+		(property "Reference" "#PWR031"
 			(at 132.08 138.43 0)
 			(effects
@@
 			(project "motor_driver"
 				(path "/1ef6600e-ea1d-4a9a-8ae5-1c3f7136836c/51484c10-a339-47e4-a28f-1fe6df54aaa5"
-					(reference "#PWR043")
+					(reference "#PWR031")
 					(unit 1)
 				)
@@
 		(dnp no)
 		(fields_autoplaced yes)
-		(property "Reference" "#PWR040"
+		(property "Reference" "#PWR028"
 			(at 124.46 101.6 0)
 			(effects
@@
 			(project "motor_driver"
 				(path "/1ef6600e-ea1d-4a9a-8ae5-1c3f7136836c/51484c10-a339-47e4-a28f-1fe6df54aaa5"
-					(reference "#PWR040")
+					(reference "#PWR028")
 					(unit 1)
 				)
@@
 		(dnp no)
 		(fields_autoplaced yes)
-		(property "Reference" "C17"
+		(property "Reference" "C16"
 			(at 162.56 88.9062 0)
 			(effects
@@
 			(project "motor_driver"
 				(path "/1ef6600e-ea1d-4a9a-8ae5-1c3f7136836c/51484c10-a339-47e4-a28f-1fe6df54aaa5"
-					(reference "C17")
+					(reference "C16")
 					(unit 1)
 				)
@@
 		(dnp no)
 		(fields_autoplaced yes)
-		(property "Reference" "#PWR044"
+		(property "Reference" "#PWR032"
 			(at 160.02 101.6 0)
 			(effects
@@
 			(project "motor_driver"
 				(path "/1ef6600e-ea1d-4a9a-8ae5-1c3f7136836c/51484c10-a339-47e4-a28f-1fe6df54aaa5"
-					(reference "#PWR044")
+					(reference "#PWR032")
 					(unit 1)
 				)
@@
 		(dnp no)
 		(fields_autoplaced yes)
-		(property "Reference" "#PWR047"
+		(property "Reference" "#PWR035"
 			(at 172.72 116.84 0)
 			(effects
@@
 			(project "motor_driver"
 				(path "/1ef6600e-ea1d-4a9a-8ae5-1c3f7136836c/51484c10-a339-47e4-a28f-1fe6df54aaa5"
-					(reference "#PWR047")
+					(reference "#PWR035")
 					(unit 1)
 				)
@@
 		(dnp no)
 		(fields_autoplaced yes)
-		(property "Reference" "#PWR042"
+		(property "Reference" "#PWR030"
 			(at 132.08 101.6 0)
 			(effects
@@
 			(project "motor_driver"
 				(path "/1ef6600e-ea1d-4a9a-8ae5-1c3f7136836c/51484c10-a339-47e4-a28f-1fe6df54aaa5"
-					(reference "#PWR042")
+					(reference "#PWR030")
 					(unit 1)
 				)
@@
 		(dnp no)
 		(fields_autoplaced yes)
-		(property "Reference" "#PWR046"
+		(property "Reference" "#PWR034"
 			(at 172.72 101.6 0)
 			(effects
@@
 			(project "motor_driver"
 				(path "/1ef6600e-ea1d-4a9a-8ae5-1c3f7136836c/51484c10-a339-47e4-a28f-1fe6df54aaa5"
-					(reference "#PWR046")
+					(reference "#PWR034")
 					(unit 1)
 				)
@@
 		(dnp no)
 		(fields_autoplaced yes)
-		(property "Reference" "C19"
+		(property "Reference" "C18"
 			(at 175.26 125.7362 0)
 			(effects
@@
 			(project "motor_driver"
 				(path "/1ef6600e-ea1d-4a9a-8ae5-1c3f7136836c/51484c10-a339-47e4-a28f-1fe6df54aaa5"
-					(reference "C19")
+					(reference "C18")
 					(unit 1)
 				)
@@
 		(dnp no)
 		(fields_autoplaced yes)
-		(property "Reference" "D4"
+		(property "Reference" "D1"
 			(at 207.01 79.0574 90)
 			(effects
@@
 			)
 		)
-		(property "Footprint" "LED_SMD:LED_0603_1608Metric_Pad1.05x0.95mm_HandSolder"
+		(property "Footprint" "LED_SMD:LED_0603_1608Metric"
 			(at 203.2 78.74 0)
 			(effects
@@
 			(project "motor_driver"
 				(path "/1ef6600e-ea1d-4a9a-8ae5-1c3f7136836c/51484c10-a339-47e4-a28f-1fe6df54aaa5"
-					(reference "D4")
+					(reference "D1")
 					(unit 1)
 				)
@@
 		(dnp no)
 		(fields_autoplaced yes)
-		(property "Reference" "U9"
+		(property "Reference" "U4"
 			(at 146.685 74.93 0)
 			(effects
@@
 			(project "motor_driver"
 				(path "/1ef6600e-ea1d-4a9a-8ae5-1c3f7136836c/51484c10-a339-47e4-a28f-1fe6df54aaa5"
-					(reference "U9")
+					(reference "U4")
 					(unit 1)
 				)
@@
 		(dnp no)
 		(fields_autoplaced yes)
-		(property "Reference" "C14"
+		(property "Reference" "C13"
 			(at 106.68 88.9062 0)
 			(effects
@@
 			(project "motor_driver"
 				(path "/1ef6600e-ea1d-4a9a-8ae5-1c3f7136836c/51484c10-a339-47e4-a28f-1fe6df54aaa5"
-					(reference "C14")
+					(reference "C13")
 					(unit 1)
 				)
@@
 		(dnp no)
 		(fields_autoplaced yes)
-		(property "Reference" "#PWR041"
+		(property "Reference" "#PWR029"
 			(at 124.46 138.43 0)
 			(effects
@@
 			(project "motor_driver"
 				(path "/1ef6600e-ea1d-4a9a-8ae5-1c3f7136836c/51484c10-a339-47e4-a28f-1fe6df54aaa5"
-					(reference "#PWR041")
+					(reference "#PWR029")
 					(unit 1)
 				)
@@
 		(dnp no)
 		(fields_autoplaced yes)
-		(property "Reference" "C18"
+		(property "Reference" "C17"
 			(at 175.26 88.9062 0)
 			(effects
@@
 			(project "motor_driver"
 				(path "/1ef6600e-ea1d-4a9a-8ae5-1c3f7136836c/51484c10-a339-47e4-a28f-1fe6df54aaa5"
-					(reference "C18")
+					(reference "C17")
 					(unit 1)
 				)
@@
 		(dnp no)
 		(fields_autoplaced yes)
-		(property "Reference" "#PWR049"
+		(property "Reference" "#PWR037"
 			(at 203.2 77.47 0)
 			(effects
@@
 			(project "motor_driver"
 				(path "/1ef6600e-ea1d-4a9a-8ae5-1c3f7136836c/51484c10-a339-47e4-a28f-1fe6df54aaa5"
-					(reference "#PWR049")
+					(reference "#PWR037")
 					(unit 1)
 				)
@@
 		(dnp no)
 		(fields_autoplaced yes)
-		(property "Reference" "#PWR048"
+		(property "Reference" "#PWR036"
 			(at 172.72 138.43 0)
 			(effects
@@
 			(project "motor_driver"
 				(path "/1ef6600e-ea1d-4a9a-8ae5-1c3f7136836c/51484c10-a339-47e4-a28f-1fe6df54aaa5"
-					(reference "#PWR048")
+					(reference "#PWR036")
 					(unit 1)
 				)
@@
 		(dnp no)
 		(fields_autoplaced yes)
-		(property "Reference" "U8"
+		(property "Reference" "U3"
 			(at 146.685 111.76 0)
 			(effects
@@
 			(project "motor_driver"
 				(path "/1ef6600e-ea1d-4a9a-8ae5-1c3f7136836c/51484c10-a339-47e4-a28f-1fe6df54aaa5"
-					(reference "U8")
+					(reference "U3")
 					(unit 1)
 				)
@@
 		(dnp no)
 		(fields_autoplaced yes)
-		(property "Reference" "#PWR045"
+		(property "Reference" "#PWR033"
 			(at 172.72 77.47 0)
 			(effects
@@
 			(project "motor_driver"
 				(path "/1ef6600e-ea1d-4a9a-8ae5-1c3f7136836c/51484c10-a339-47e4-a28f-1fe6df54aaa5"
-					(reference "#PWR045")
+					(reference "#PWR033")
 					(unit 1)
 				)
@@
 		(dnp no)
 		(fields_autoplaced yes)
-		(property "Reference" "#PWR050"
+		(property "Reference" "#PWR038"
 			(at 203.2 101.6 0)
 			(effects
@@
 			(project "motor_driver"
 				(path "/1ef6600e-ea1d-4a9a-8ae5-1c3f7136836c/51484c10-a339-47e4-a28f-1fe6df54aaa5"
-					(reference "#PWR050")
+					(reference "#PWR038")
 					(unit 1)
 				)
@@
 		(dnp no)
 		(fields_autoplaced yes)
-		(property "Reference" "#PWR038"
+		(property "Reference" "#PWR026"
 			(at 104.14 77.47 0)
 			(effects
@@
 			(project "motor_driver"
 				(path "/1ef6600e-ea1d-4a9a-8ae5-1c3f7136836c/51484c10-a339-47e4-a28f-1fe6df54aaa5"
-					(reference "#PWR038")
+					(reference "#PWR026")
 					(unit 1)
 				)
@@
 		(dnp no)
 		(fields_autoplaced yes)
-		(property "Reference" "#PWR039"
+		(property "Reference" "#PWR027"
 			(at 104.14 101.6 0)
 			(effects
@@
 			(project "motor_driver"
 				(path "/1ef6600e-ea1d-4a9a-8ae5-1c3f7136836c/51484c10-a339-47e4-a28f-1fe6df54aaa5"
-					(reference "#PWR039")
+					(reference "#PWR027")
 					(unit 1)
 				)
@@
 		(dnp no)
 		(fields_autoplaced yes)
-		(property "Reference" "R13"
+		(property "Reference" "R10"
 			(at 205.74 87.6299 0)
 			(effects
@@
 			)
 		)
-		(property "Footprint" "Resistor_SMD:R_0402_1005Metric_Pad0.72x0.64mm_HandSolder"
+		(property "Footprint" "Resistor_SMD:R_0603_1608Metric_Pad0.98x0.95mm_HandSolder"
 			(at 203.2 88.9 0)
 			(effects
@@
 			(project "motor_driver"
 				(path "/1ef6600e-ea1d-4a9a-8ae5-1c3f7136836c/51484c10-a339-47e4-a28f-1fe6df54aaa5"
-					(reference "R13")
+					(reference "R10")
 					(unit 1)
 				)
@@
 		(dnp no)
 		(fields_autoplaced yes)
-		(property "Reference" "C16"
+		(property "Reference" "C15"
 			(at 127 125.7362 0)
 			(effects
@@
 			(project "motor_driver"
 				(path "/1ef6600e-ea1d-4a9a-8ae5-1c3f7136836c/51484c10-a339-47e4-a28f-1fe6df54aaa5"
-					(reference "C16")
+					(reference "C15")
 					(unit 1)
 				)
@@
 		(dnp no)
 		(fields_autoplaced yes)
-		(property "Reference" "C15"
+		(property "Reference" "C14"
 			(at 127 88.9062 0)
 			(effects
@@
 			(project "motor_driver"
 				(path "/1ef6600e-ea1d-4a9a-8ae5-1c3f7136836c/51484c10-a339-47e4-a28f-1fe6df54aaa5"
-					(reference "C15")
-					(unit 1)
-				)
+					(reference "C14")
+					(unit 1)
+				)

Commit message: perf: update motor driver pdb
Parts:
- added D8: LED, LED_SMD:LED_0603_1608Metric, symbol Device:LED
- added R24: 1k, Resistor_SMD:R_0603_1608Metric_Pad0.98x0.95mm_HandSolder, symbol Device:R_Small
Connections:
- net +3.3V: now also R10.1; no longer D1.2 (A)
- net +3.3VA: now also R24.1
- net GND: now also D1.1 (K), D8.1 (K); no longer R10.2
- new net: D1.2 (A), R10.2
- new net: D8.2 (A), R24.2
Other:
- moved on the sheet: D1, R10

Commit message: feat: add additional CAN connetctor
Parts:
- renumbered D8 to D2, R24 to R11
Changed lines of the file:
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@@
 		(dnp no)
 		(fields_autoplaced yes)
-		(property "Reference" "#PWR075"
+		(property "Reference" "#PWR039"
 			(at 203.2 116.84 0)
 			(effects
@@
 			(project "motor_driver"
 				(path "/1ef6600e-ea1d-4a9a-8ae5-1c3f7136836c/51484c10-a339-47e4-a28f-1fe6df54aaa5"
-					(reference "#PWR075")
+					(reference "#PWR039")
 					(unit 1)
 				)
@@
 		(dnp no)
 		(fields_autoplaced yes)
-		(property "Reference" "#PWR077"
+		(property "Reference" "#PWR040"
 			(at 203.2 140.97 0)
 			(effects
@@
 			(project "motor_driver"
 				(path "/1ef6600e-ea1d-4a9a-8ae5-1c3f7136836c/51484c10-a339-47e4-a28f-1fe6df54aaa5"
-					(reference "#PWR077")
+					(reference "#PWR040")
 					(unit 1)
 				)
@@
 		(dnp no)
 		(fields_autoplaced yes)
-		(property "Reference" "D8"
+		(property "Reference" "D2"
 			(at 207.01 127.3174 90)
 			(effects
@@
 			(project "motor_driver"
 				(path "/1ef6600e-ea1d-4a9a-8ae5-1c3f7136836c/51484c10-a339-47e4-a28f-1fe6df54aaa5"
-					(reference "D8")
+					(reference "D2")
 					(unit 1)
 				)
@@
 		(dnp no)
 		(fields_autoplaced yes)
-		(property "Reference" "R24"
+		(property "Reference" "R11"
 			(at 205.74 119.3799 0)
 			(effects
@@
 			(project "motor_driver"
 				(path "/1ef6600e-ea1d-4a9a-8ae5-1c3f7136836c/51484c10-a339-47e4-a28f-1fe6df54aaa5"
-					(reference "R24")
-					(unit 1)
-				)
+					(reference "R11")
+					(unit 1)
+				)
